File: pcbs/assemble_l/bias.kicad_sch (KiCad schematic)
At the start: 48 parts, among them J1 TRRS_MJ-4PP-9, J2 Conn_01x02, SW1 SW_Push, SW10 SW_Push, SW11 SW_Push, SW12 SW_Push, SW13 SW_Push, SW14 SW_Push, SW15 SW_Push, SW16 SW_Push, SW17 SW_Push, SW18 SW_Push, SW19 SW_Push, SW2 SW_Push, SW20 SW_Push, SW21 SW_Push, SW22 SW_Push, SW23 SW_Push, SW3 SW_Push, SW4 SW_Push, SW5 SW_Push, SW6 SW_Push, SW7 SW_Push, SW8 SW_Push, SW9 SW_Push, U1 Micon_BLEMicroPro

Commit message: Reorganize PCB project files and add edge cut DXFs
Parts:
- J2: footprint kbd_Parts:Battery_BMP_2pin -> kbd_Parts:Battery_2pin
Changed lines of the file:
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@@
 			)
 		)
-		(property "Footprint" "kbd_Parts:Battery_BMP_2pin"
+		(property "Footprint" "kbd_Parts:Battery_2pin"
 			(at 87.63 104.14 0)
 			(effects
